Commit message: modified for custom 4-axis robot

File: annin_ar4_description/urdf/ar.ros2_control.xacro (robot description, xacro)
@@ -83,5 +83,5 @@
         <param name="position_offset">${joint_offset_parameters['joint_4']}</param>
       </joint>
-      <joint name="${tf_prefix}joint_5">
+<!--       <joint name="${tf_prefix}joint_5">
         <command_interface name="position">
           <param name="min">${robot_parameters['j5_limit_min']}</param>
@@ -110,5 +110,5 @@
         </state_interface>
         <param name="position_offset">${joint_offset_parameters['joint_6']}</param>
-      </joint>
+      </joint> -->
     </ros2_control>
   </xacro:macro>

File: annin_ar4_moveit_config/config/ar.srdf.xacro (robot description, xacro)
@@ -1,11 +1,11 @@
 <?xml version="1.0" encoding="UTF-8"?>
-<robot xmlns:xacro="http://wiki.ros.org/xacro" name="$(arg name)">
+<robot xmlns:xacro="http://wiki.ros.org/xacro" name="ar">
   <xacro:arg name="include_gripper" default="true"/>
   <xacro:arg name="tf_prefix" default="" />
-  <xacro:include filename="$(find annin_ar4_moveit_config)/srdf/ar_macro.srdf.xacro"/>
+  <xacro:include filename="$(find annin_ar4_moveit_config)/config/ar_macro.srdf.xacro"/>
   <xacro:ar_srdf tf_prefix="$(arg tf_prefix)"/>
-  <xacro:if value="$(arg include_gripper)">
+<!--   <xacro:if value="$(arg include_gripper)">
     <xacro:include filename="$(find annin_ar4_moveit_config)/srdf/ar_gripper_macro.srdf.xacro"/>
     <xacro:ar_gripper_srdf tf_prefix="$(arg tf_prefix)"/>
-  </xacro:if>
+  </xacro:if> -->
 </robot>

File: annin_ar4_moveit_config/config/ar.urdf.xacro (robot description, xacro)
@@ -1,10 +1,11 @@
 <?xml version="1.0"?>
-<robot xmlns:xacro="http://wiki.ros.org/xacro" name="$(arg ar_model)">
-  <xacro:include filename="$(find annin_ar4_description)/urdf/ar_macro.xacro"/>
-  <xacro:include filename="$(find annin_ar4_description)/urdf/ar_gripper_macro.xacro"/>
+<robot xmlns:xacro="http://wiki.ros.org/xacro" name="ar">
+  <xacro:include filename="$(find sketch_bot_support)/urdf/sketch_bot_macro.xacro"/>
+  <!-- <xacro:include filename="$(find annin_ar4_description)/urdf/ar_gripper_macro.xacro"/> -->
   <xacro:include filename="$(find annin_ar4_description)/urdf/ar.ros2_control.xacro"/>
-  <xacro:include filename="$(find annin_ar4_description)/urdf/ar_gripper.ros2_control.xacro"/>
+  <!-- <xacro:include filename="$(find annin_ar4_description)/urdf/ar_gripper.ros2_control.xacro"/> -->
   <xacro:arg name="tf_prefix" default="" />
-  <link name="world" />
+  <xacro:arg name="ar_model" default="mk3" />
+<!--   <link name="world" />
   <xacro:ar_robot
     tf_prefix="$(arg tf_prefix)"
@@ -13,9 +14,10 @@
   >
     <origin xyz="0 0 0" rpy="0 0 0" />
-  </xacro:ar_robot>
-  <xacro:ar_gripper
+  </xacro:ar_robot> -->
+  <xacro:sketch_bot prefix="$(arg tf_prefix)"/>
+<!--   <xacro:ar_gripper
     tf_prefix="$(arg tf_prefix)"
     parent="$(arg tf_prefix)ee_link"
-  />
+  /> -->
   <xacro:ar_ros2_control
     ar_model="$(arg ar_model)"
@@ -28,5 +30,5 @@
     tf_prefix="$(arg tf_prefix)"
   />
-  <xacro:ar_gripper_ros2_control
+<!--   <xacro:ar_gripper_ros2_control
     name="ARGripperFakeSystem"
     plugin_name="mock_components/GenericSystem"
@@ -34,4 +36,4 @@
     driver_parameters_file="$(find annin_ar4_driver)/config/gripper_driver.yaml"
     tf_prefix="$(arg tf_prefix)"
-  />
+  /> -->
 </robot>

File: annin_ar4_moveit_config/config/ar_macro.srdf.xacro (robot description, xacro)
@@ -11,7 +11,7 @@
       <joint name="${tf_prefix}joint_3" />
       <joint name="${tf_prefix}joint_4" />
-      <joint name="${tf_prefix}joint_5" />
+<!--       <joint name="${tf_prefix}joint_5" />
       <joint name="${tf_prefix}joint_6" />
-      <joint name="${tf_prefix}ee_joint"/>
+      <joint name="${tf_prefix}ee_joint"/> -->
     </group>
     <group_state name="home" group="ar_manipulator">
@@ -20,6 +20,6 @@
       <joint name="${tf_prefix}joint_3" value="0" />
       <joint name="${tf_prefix}joint_4" value="0" />
-      <joint name="${tf_prefix}joint_5" value="0" />
-      <joint name="${tf_prefix}joint_6" value="0" />
+<!--       <joint name="${tf_prefix}joint_5" value="0" />
+      <joint name="${tf_prefix}joint_6" value="0" /> -->
     </group_state>
     <group_state name="upright" group="ar_manipulator">
@@ -28,6 +28,6 @@
       <joint name="${tf_prefix}joint_3" value="-1.4" />
       <joint name="${tf_prefix}joint_4" value="0" />
-      <joint name="${tf_prefix}joint_5" value="0" />
-      <joint name="${tf_prefix}joint_6" value="0" />
+<!--       <joint name="${tf_prefix}joint_5" value="0" />
+      <joint name="${tf_prefix}joint_6" value="0" /> -->
     </group_state>
     <disable_collisions link1="${tf_prefix}base_link" link2="${tf_prefix}link_1" reason="Adjacent" />
@@ -36,8 +36,8 @@
     <disable_collisions link1="${tf_prefix}link_2" link2="${tf_prefix}link_3" reason="Adjacent" />
     <disable_collisions link1="${tf_prefix}link_3" link2="${tf_prefix}link_4" reason="Adjacent" />
-    <disable_collisions link1="${tf_prefix}link_3" link2="${tf_prefix}link_5" reason="Never" />
-    <disable_collisions link1="${tf_prefix}link_3" link2="${tf_prefix}link_6" reason="Never" />
-    <disable_collisions link1="${tf_prefix}link_4" link2="${tf_prefix}link_5" reason="Adjacent" />
-    <disable_collisions link1="${tf_prefix}link_5" link2="${tf_prefix}link_6" reason="Adjacent" />
+    <!-- <disable_collisions link1="${tf_prefix}link_3" link2="${tf_prefix}link_5" reason="Never" /> -->
+    <!-- <disable_collisions link1="${tf_prefix}link_3" link2="${tf_prefix}link_6" reason="Never" /> -->
+    <!-- <disable_collisions link1="${tf_prefix}link_4" link2="${tf_prefix}link_5" reason="Adjacent" /> -->
+    <!-- <disable_collisions link1="${tf_prefix}link_5" link2="${tf_prefix}link_6" reason="Adjacent" /> -->
   </xacro:macro>
 </robot>
