Commit message: adapted driver to work with 4-dof custom robot

File: annin_ar4_driver/urdf/ar.urdf.xacro (robot description, xacro)
@@ -3,10 +3,11 @@
   <xacro:arg name="serial_port" default="/dev/ttyACM0"/>
   <xacro:arg name="arduino_serial_port" default="/dev/ttyUSB0"/>
-  <xacro:arg name="calibrate" default="True"/>
+  <xacro:arg name="calibrate" default="false"/>
   <xacro:arg name="tf_prefix" default="" />
-  <xacro:arg name="include_gripper" default="true"/>
-  <xacro:include filename="$(find annin_ar4_description)/urdf/ar_macro.xacro"/>
+  <xacro:arg name="include_gripper" default="false"/>
+  <xacro:include filename="$(find sketch_bot_support)/urdf/sketch_bot_macro.xacro"/>
   <xacro:include filename="$(find annin_ar4_description)/urdf/ar.ros2_control.xacro"/>
-  <link name="world" />
+  <xacro:sketch_bot prefix=""/>
+  <!-- <link name="world" />
   <xacro:ar_robot
     tf_prefix="$(arg tf_prefix)"
@@ -15,5 +16,5 @@
   >
     <origin xyz="0 0 0" rpy="0 0 0" />
-  </xacro:ar_robot>
+  </xacro:ar_robot> -->
   <xacro:ar_ros2_control
     ar_model="$(arg ar_model)"
@@ -26,5 +27,5 @@
     tf_prefix="$(arg tf_prefix)"
   />
-  <xacro:if value="$(arg include_gripper)">
+  <!-- <xacro:if value="$(arg include_gripper)">
     <xacro:include filename="$(find annin_ar4_description)/urdf/ar_gripper_macro.xacro"/>
     <xacro:include filename="$(find annin_ar4_description)/urdf/ar_gripper.ros2_control.xacro"/>
@@ -40,4 +41,4 @@
       tf_prefix="$(arg tf_prefix)"
     />
-  </xacro:if>
+  </xacro:if> -->
 </robot>
